File: electronics/audio_ver1_0/untitled.brd (EAGLE design)
At the start: 70 x 40 mm, 45 parts, among them IC1 PCM2704DBG4, IC2 NJM2845DL1-33-TE1, IC3 2N7002K, IC4 UPA2735GR-E2-AX, Y1 FA-238V_12.0000MB-K3

Commit message: push audio_ver1_0
Parts:
- A_C2, A_C4: value (none) -> 47μ
- C11: value (none) -> 10μ
- C14: value 50PK4R7MEFC5X11 -> 4.7μ
- C18: value (none) -> 0.047μ
Changed lines of the file:
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@@
 <attribute name="VALUE" x="12.827" y="21.971" size="1.27" layer="27" rot="R180"/>
 </element>
-<element name="C14" library="SamacSys_Parts" package="CAPPRD200W50D525H1100" value="50PK4R7MEFC5X11" x="39.346" y="25.86" smashed="yes">
+<element name="C14" library="SamacSys_Parts" package="CAPPRD200W50D525H1100" value="4.7μ" x="39.346" y="25.86" smashed="yes">
 <attribute name="DESCRIPTION" value="Rubycon Aluminium Electrolytic Capacitor PK Series 50V dc 4.7uF, Through Hole Electrolytic, +/-20% +85C" x="62.206" y="-14.78" size="1.778" layer="27" display="off"/>
 <attribute name="HEIGHT" value="11mm" x="62.206" y="-14.78" size="1.778" layer="27" display="off"/>
@@
 <attribute name="VALUE" x="51.181" y="16.891" size="1.27" layer="27"/>
 </element>
-<element name="C18" library="50F2D473J" package="50F2D473J" value="" x="26.416" y="22.352" smashed="yes" rot="R270"/>
+<element name="C18" library="50F2D473J" package="50F2D473J" value="0.047μ" x="26.416" y="22.352" smashed="yes" rot="R270"/>
 <element name="C2" library="rcl" library_urn="urn:adsk.eagle:library:334" package="C0603" package3d_urn="urn:adsk.eagle:package:23616/2" value="0.1μ" x="35.136" y="18.48" smashed="yes">
 <attribute name="NAME" x="31.453" y="17.591" size="1.27" layer="25"/>
@@
 <attribute name="VALUE" x="2.286" y="7.62" size="1.27" layer="27" align="center"/>
 </element>
-<element name="A_C2" library="UFG1E470MEM" package="UFG1E470MEM" value="" x="62.484" y="17.526" smashed="yes">
+<element name="A_C2" library="UFG1E470MEM" package="UFG1E470MEM" value="47μ" x="62.484" y="17.526" smashed="yes">
 <attribute name="NAME" x="57.404" y="20.066" size="1.27" layer="25"/>
 </element>
-<element name="A_C4" library="UFG1E470MEM" package="UFG1E470MEM" value="" x="57.912" y="32.004" smashed="yes">
+<element name="A_C4" library="UFG1E470MEM" package="UFG1E470MEM" value="47μ" x="57.912" y="32.004" smashed="yes">
 <attribute name="NAME" x="52.832" y="34.544" size="1.27" layer="25"/>
 </element>
-<element name="C11" library="50F2D473J" package="50F2D473J" value="" x="42.958" y="37.576" smashed="yes" rot="R180"/>
+<element name="C11" library="50F2D473J" package="50F2D473J" value="10μ" x="42.958" y="37.576" smashed="yes" rot="R180"/>
 </elements>
 <signals>
