File: electronics/audio_ver1_0/untitled.sch (EAGLE design)
At the start: 45 parts, among them IC1 PCM2704DBG4, IC2 NJM2845DL1-33-TE1, IC3 2N7002K, IC4 UPA2735GR-E2-AX, J1 USB2066-05-RBHM-15-STB-00-00-A, Y1 FA-238V_12.0000MB-K3

Commit message: push audio_ver1_0
Parts:
- A_C2, A_C4: value (none) -> 47μ
- C11: value (none) -> 10μ
- C14: value 50PK4R7MEFC5X11 -> 4.7μ
- C18: value (none) -> 0.047μ
Changed lines of the file:
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@@
 <part name="GND23" library="supply1" library_urn="urn:adsk.eagle:library:371" deviceset="GND" device=""/>
 <part name="VR1" library="SamacSys_Parts" deviceset="TSR-3386T-EY5-103TR" device=""/>
-<part name="C14" library="SamacSys_Parts" deviceset="50PK4R7MEFC5X11" device=""/>
+<part name="C14" library="SamacSys_Parts" deviceset="50PK4R7MEFC5X11" device="" value="4.7μ"/>
 <part name="C16" library="SamacSys_Parts" deviceset="50PK10MEFC5X11" device="" value="10μ"/>
 <part name="C17" library="rcl" library_urn="urn:adsk.eagle:library:334" deviceset="C-EU" device="C0603" package3d_urn="urn:adsk.eagle:package:23616/2" value="0.1μ"/>
@@
 <part name="J1" library="SamacSys_Parts" deviceset="USB2066-05-RBHM-15-STB-00-00-A" device="" value=""/>
 <part name="GND25" library="supply1" library_urn="urn:adsk.eagle:library:371" deviceset="GND" device=""/>
-<part name="C18" library="50F2D473J" deviceset="50F2D473J" device=""/>
+<part name="C18" library="50F2D473J" deviceset="50F2D473J" device="" value="0.047μ"/>
 <part name="GND21" library="supply1" library_urn="urn:adsk.eagle:library:371" deviceset="GND" device=""/>
 <part name="Z1" library="SamacSys_Parts" deviceset="UDZVTE-175.1B" device=""/>
 <part name="GND1" library="supply1" library_urn="urn:adsk.eagle:library:371" deviceset="GND" device=""/>
-<part name="A_C2" library="UFG1E470MEM" deviceset="UFG1E470MEM" device=""/>
-<part name="A_C4" library="UFG1E470MEM" deviceset="UFG1E470MEM" device=""/>
-<part name="C11" library="50F2D473J" deviceset="50F2D473J" device=""/>
+<part name="A_C2" library="UFG1E470MEM" deviceset="UFG1E470MEM" device="" value="47μ"/>
+<part name="A_C4" library="UFG1E470MEM" deviceset="UFG1E470MEM" device="" value="47μ"/>
+<part name="C11" library="50F2D473J" deviceset="50F2D473J" device="" value="10μ"/>
 <part name="P+1" library="supply1" library_urn="urn:adsk.eagle:library:371" deviceset="V+" device="" value="AVCC"/>
 <part name="P+6" library="supply1" library_urn="urn:adsk.eagle:library:371" deviceset="V+" device="" value="AVCC"/>
